File: Projects/RaspberryPi-HAT/RaspberryPi-HAT.kicad_sch (KiCad schematic)
At the start: 6 parts, among them J1 GPIO, U1 CAT24C256

Commit message: Fix v6 net names
Connections:
- net GPIO[10]/SPI0.MOSI renamed GPIO10/SPI0.MOSI
- net GPIO[11]/SPI0.SCLK renamed GPIO11/SPI0.SCLK
- net GPIO[12]/PWM0 renamed GPIO12/PWM0
- net GPIO[13]/PWM1 renamed GPIO13/PWM1
- net GPIO[14]/TXD0 renamed GPIO14/TXD0
- net GPIO[15]/RXD0 renamed GPIO15/RXD0
- net GPIO[16] renamed GPIO16
- net GPIO[17] renamed GPIO17
- net GPIO[18]/PCM.CLK renamed GPIO18/PCM.CLK
- net GPIO[19]/PCM.FS renamed GPIO19/PCM.FS
- net GPIO[20]/PCM.DIN renamed GPIO20/PCM.DIN
- net GPIO[21]/PCM.DOUT renamed GPIO21/PCM.DOUT
- net GPIO[22] renamed GPIO22
- net GPIO[23] renamed GPIO23
- net GPIO[24] renamed GPIO24
- net GPIO[25] renamed GPIO25
- net GPIO[26] renamed GPIO26
- net GPIO[27] renamed GPIO27
- net GPIO[2]/SDA1 renamed GPIO2/SDA1
- net GPIO[3]/SCL1 renamed GPIO3/SCL1
- net GPIO[4]/GPCLK0 renamed GPIO4/GPCLK0
- net GPIO[5] renamed GPIO5
- net GPIO[6] renamed GPIO6
- net GPIO[7]/SPI0.CE1 renamed GPIO7/SPI0.CE1
- net GPIO[8]/SPI0.CE0 renamed GPIO8/SPI0.CE0
- net GPIO[9]/SPI0.MISO renamed GPIO9/SPI0.MISO
Changed lines of the file:
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@@
     (effects (font (size 1.27 1.27)) (justify left bottom))
   )
-  (label "GPIO[6]" (at 31.75 66.04 0)
+  (label "GPIO6" (at 31.75 66.04 0)
     (effects (font (size 1.27 1.27)) (justify left bottom))
   )
@@
     (effects (font (size 1.27 1.27)) (justify right bottom))
   )
-  (label "GPIO[5]" (at 31.75 63.5 0)
+  (label "GPIO5" (at 31.75 63.5 0)
     (effects (font (size 1.27 1.27)) (justify left bottom))
   )
-  (label "GPIO[21]{slash}PCM.DOUT" (at 100.33 76.2 180)
+  (label "GPIO21{slash}PCM.DOUT" (at 100.33 76.2 180)
     (effects (font (size 1.27 1.27)) (justify right bottom))
   )
-  (label "GPIO[19]{slash}PCM.FS" (at 31.75 71.12 0)
+  (label "GPIO19{slash}PCM.FS" (at 31.75 71.12 0)
     (effects (font (size 1.27 1.27)) (justify left bottom))
   )
-  (label "GPIO[10]{slash}SPI0.MOSI" (at 31.75 50.8 0)
+  (label "GPIO10{slash}SPI0.MOSI" (at 31.75 50.8 0)
     (effects (font (size 1.27 1.27)) (justify left bottom))
   )
-  (label "GPIO[9]{slash}SPI0.MISO" (at 31.75 53.34 0)
+  (label "GPIO9{slash}SPI0.MISO" (at 31.75 53.34 0)
     (effects (font (size 1.27 1.27)) (justify left bottom))
   )
-  (label "GPIO[23]" (at 100.33 45.72 180)
+  (label "GPIO23" (at 100.33 45.72 180)
     (effects (font (size 1.27 1.27)) (justify right bottom))
   )
-  (label "GPIO[4]{slash}GPCLK0" (at 31.75 35.56 0)
+  (label "GPIO4{slash}GPCLK0" (at 31.75 35.56 0)
     (effects (font (size 1.27 1.27)) (justify left bottom))
   )
-  (label "GPIO[27]" (at 31.75 43.18 0)
+  (label "GPIO27" (at 31.75 43.18 0)
     (effects (font (size 1.27 1.27)) (justify left bottom))
   )
-  (label "GPIO[26]" (at 31.75 73.66 0)
+  (label "GPIO26" (at 31.75 73.66 0)
     (effects (font (size 1.27 1.27)) (justify left bottom))
   )
-  (label "GPIO[14]{slash}TXD0" (at 100.33 35.56 180)
+  (label "GPIO14{slash}TXD0" (at 100.33 35.56 180)
     (effects (font (size 1.27 1.27)) (justify right bottom))
   )
-  (label "GPIO[8]{slash}SPI0.CE0" (at 100.33 55.88 180)
+  (label "GPIO8{slash}SPI0.CE0" (at 100.33 55.88 180)
     (effects (font (size 1.27 1.27)) (justify right bottom))
   )
-  (label "GPIO[15]{slash}RXD0" (at 100.33 38.1 180)
+  (label "GPIO15{slash}RXD0" (at 100.33 38.1 180)
     (effects (font (size 1.27 1.27)) (justify right bottom))
   )
-  (label "GPIO[16]" (at 100.33 71.12 180)
+  (label "GPIO16" (at 100.33 71.12 180)
     (effects (font (size 1.27 1.27)) (justify right bottom))
   )
-  (label "GPIO[22]" (at 31.75 45.72 0)
+  (label "GPIO22" (at 31.75 45.72 0)
     (effects (font (size 1.27 1.27)) (justify left bottom))
   )
-  (label "GPIO[2]{slash}SDA1" (at 31.75 30.48 0)
+  (label "GPIO2{slash}SDA1" (at 31.75 30.48 0)
     (effects (font (size 1.27 1.27)) (justify left bottom))
   )
-  (label "GPIO[17]" (at 31.75 40.64 0)
+  (label "GPIO17" (at 31.75 40.64 0)
     (effects (font (size 1.27 1.27)) (justify left bottom))
   )
-  (label "GPIO[25]" (at 100.33 53.34 180)
+  (label "GPIO25" (at 100.33 53.34 180)
     (effects (font (size 1.27 1.27)) (justify right bottom))
   )
-  (label "GPIO[3]{slash}SCL1" (at 31.75 33.02 0)
+  (label "GPIO3{slash}SCL1" (at 31.75 33.02 0)
     (effects (font (size 1.27 1.27)) (justify left bottom))
   )
-  (label "GPIO[18]{slash}PCM.CLK" (at 100.33 40.64 180)
+  (label "GPIO18{slash}PCM.CLK" (at 100.33 40.64 180)
     (effects (font (size 1.27 1.27)) (justify right bottom))
   )
-  (label "GPIO[12]{slash}PWM0" (at 100.33 66.04 180)
+  (label "GPIO12{slash}PWM0" (at 100.33 66.04 180)
     (effects (font (size 1.27 1.27)) (justify right bottom))
   )
-  (label "GPIO[13]{slash}PWM1" (at 31.75 68.58 0)
+  (label "GPIO13{slash}PWM1" (at 31.75 68.58 0)
     (effects (font (size 1.27 1.27)) (justify left bottom))
   )
-  (label "GPIO[20]{slash}PCM.DIN" (at 100.33 73.66 180)
+  (label "GPIO20{slash}PCM.DIN" (at 100.33 73.66 180)
     (effects (font (size 1.27 1.27)) (justify right bottom))
   )
-  (label "GPIO[24]" (at 100.33 48.26 180)
+  (label "GPIO24" (at 100.33 48.26 180)
     (effects (font (size 1.27 1.27)) (justify right bottom))
   )
-  (label "GPIO[7]{slash}SPI0.CE1" (at 100.33 58.42 180)
+  (label "GPIO7{slash}SPI0.CE1" (at 100.33 58.42 180)
     (effects (font (size 1.27 1.27)) (justify right bottom))
   )
@@
     (effects (font (size 1.27 1.27)) (justify right bottom))
   )
-  (label "GPIO[11]{slash}SPI0.SCLK" (at 31.75 55.88 0)
+  (label "GPIO11{slash}SPI0.SCLK" (at 31.75 55.88 0)
     (effects (font (size 1.27 1.27)) (justify left bottom))
   )
