File: Projects/TI-LaunchPad-BoosterPack-20pin/TI-LaunchPad-BoosterPack-20pin.kicad_pcb (KiCad board)
At the start: 2 copper layers, 50.8 x 34.3 mm, 3 parts, among them J1 Conn_01x10, J2 Conn_01x10

Commit message: Fix v6 net names
Connections:
- net /*D[19] renamed /*D19
- net /D[10]/SDA renamed /D10/SDA
- net /D[11] renamed /D11
- net /D[12]/SPI.CS renamed /D12/SPI.CS
- net /D[13]/SPI.CS renamed /D13/SPI.CS
- net /D[14]/SPI.MISO renamed /D14/SPI.MISO
- net /D[15]/SPI.MOSI renamed /D15/SPI.MOSI
- net /D[17] renamed /D17
- net /D[18]/SPI.CS renamed /D18/SPI.CS
- net /D[2]/A renamed /D2/A
- net /D[3]/UART.RX renamed /D3/UART.RX
- net /D[4]/UART.TX renamed /D4/UART.TX
- net /D[5] renamed /D5
- net /D[6]/A renamed /D6/A
- net /D[7]/SPI.CLK renamed /D7/SPI.CLK
- net /D[8] renamed /D8
- net /D[9]/SCL renamed /D9/SCL
- net /RST/D[16] renamed /RST/D16
Changed lines of the file:
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@@
   )
   (net 0 "")
-  (net 1 "/D[10]{slash}SDA")
-  (net 2 "/D[9]{slash}SCL")
-  (net 3 "/D[8]")
-  (net 4 "/D[7]{slash}SPI.CLK")
-  (net 5 "/D[6]{slash}A")
-  (net 6 "/D[5]")
-  (net 7 "/D[4]{slash}UART.TX")
-  (net 8 "/D[3]{slash}UART.RX")
-  (net 9 "/D[2]{slash}A")
+  (net 1 "/D2{slash}A")
+  (net 2 "/D3{slash}UART.RX")
+  (net 3 "/D4{slash}UART.TX")
+  (net 4 "/D5")
+  (net 5 "/D6{slash}A")
+  (net 6 "/D7{slash}SPI.CLK")
+  (net 7 "/D8")
+  (net 8 "/D9{slash}SCL")
+  (net 9 "/D10{slash}SDA")
   (net 10 "+3V3")
-  (net 11 "/D[11]")
-  (net 12 "/D[12]{slash}SPI.CS")
-  (net 13 "/D[13]{slash}SPI.CS")
-  (net 14 "/D[14]{slash}SPI.MISO")
-  (net 15 "/D[15]{slash}SPI.MOSI")
-  (net 16 "/RST{slash}D[16]")
-  (net 17 "/D[17]")
-  (net 18 "/D[18]{slash}SPI.CS")
-  (net 19 "/*D[19]")
+  (net 11 "/*D19")
+  (net 12 "/D18{slash}SPI.CS")
+  (net 13 "/D17")
+  (net 14 "/RST{slash}D16")
+  (net 15 "/D15{slash}SPI.MOSI")
+  (net 16 "/D14{slash}SPI.MISO")
+  (net 17 "/D13{slash}SPI.CS")
+  (net 18 "/D12{slash}SPI.CS")
+  (net 19 "/D11")
   (net 20 "GND")
   (footprint "Connector_PinSocket_2.54mm:PinSocket_1x10_P2.54mm_Vertical" (layer "B.Cu")
@@
       (net 10 "+3V3") (pinfunction "Pin_1") (pintype "passive"))
     (pad "2" thru_hole oval locked (at 0 -2.54 180) (size 1.7 1.7) (drill 1) (layers *.Cu *.Mask)
-      (net 9 "/D[2]{slash}A") (pinfunction "Pin_2") (pintype "passive"))
+      (net 1 "/D2{slash}A") (pinfunction "Pin_2") (pintype "passive"))
     (pad "3" thru_hole oval locked (at 0 -5.08 180) (size 1.7 1.7) (drill 1) (layers *.Cu *.Mask)
-      (net 8 "/D[3]{slash}UART.RX") (pinfunction "Pin_3") (pintype "passive"))
+      (net 2 "/D3{slash}UART.RX") (pinfunction "Pin_3") (pintype "passive"))
     (pad "4" thru_hole oval locked (at 0 -7.62 180) (size 1.7 1.7) (drill 1) (layers *.Cu *.Mask)
-      (net 7 "/D[4]{slash}UART.TX") (pinfunction "Pin_4") (pintype "passive"))
+      (net 3 "/D4{slash}UART.TX") (pinfunction "Pin_4") (pintype "passive"))
     (pad "5" thru_hole oval locked (at 0 -10.16 180) (size 1.7 1.7) (drill 1) (layers *.Cu *.Mask)
-      (net 6 "/D[5]") (pinfunction "Pin_5") (pintype "passive"))
+      (net 4 "/D5") (pinfunction "Pin_5") (pintype "passive"))
     (pad "6" thru_hole oval locked (at 0 -12.7 180) (size 1.7 1.7) (drill 1) (layers *.Cu *.Mask)
-      (net 5 "/D[6]{slash}A") (pinfunction "Pin_6") (pintype "passive"))
+      (net 5 "/D6{slash}A") (pinfunction "Pin_6") (pintype "passive"))
     (pad "7" thru_hole oval locked (at 0 -15.24 180) (size 1.7 1.7) (drill 1) (layers *.Cu *.Mask)
-      (net 4 "/D[7]{slash}SPI.CLK") (pinfunction "Pin_7") (pintype "passive"))
+      (net 6 "/D7{slash}SPI.CLK") (pinfunction "Pin_7") (pintype "passive"))
     (pad "8" thru_hole oval locked (at 0 -17.78 180) (size 1.7 1.7) (drill 1) (layers *.Cu *.Mask)
-      (net 3 "/D[8]") (pinfunction "Pin_8") (pintype "passive"))
+      (net 7 "/D8") (pinfunction "Pin_8") (pintype "passive"))
     (pad "9" thru_hole oval locked (at 0 -20.32 180) (size 1.7 1.7) (drill 1) (layers *.Cu *.Mask)
-      (net 2 "/D[9]{slash}SCL") (pinfunction "Pin_9") (pintype "passive"))
+      (net 8 "/D9{slash}SCL") (pinfunction "Pin_9") (pintype "passive"))
     (pad "10" thru_hole oval locked (at 0 -22.86 180) (size 1.7 1.7) (drill 1) (layers *.Cu *.Mask)
-      (net 1 "/D[10]{slash}SDA") (pinfunction "Pin_10") (pintype "passive"))
+      (net 9 "/D10{slash}SDA") (pinfunction "Pin_10") (pintype "passive"))
     (model "${KICAD6_3DMODEL_DIR}/Connector_PinSocket_2.54mm.3dshapes/PinSocket_1x10_P2.54mm_Vertical.wrl"
       (offset (xyz 0 0 0))
@@
       (net 20 "GND") (pinfunction "Pin_1") (pintype "passive"))
     (pad "2" thru_hole oval locked (at 0 -2.54 180) (size 1.7 1.7) (drill 1) (layers *.Cu *.Mask)
-      (net 19 "/*D[19]") (pinfunction "Pin_2") (pintype "passive"))
+      (net 11 "/*D19") (pinfunction "Pin_2") (pintype "passive"))
     (pad "3" thru_hole oval locked (at 0 -5.08 180) (size 1.7 1.7) (drill 1) (layers *.Cu *.Mask)
-      (net 18 "/D[18]{slash}SPI.CS") (pinfunction "Pin_3") (pintype "passive"))
+      (net 12 "/D18{slash}SPI.CS") (pinfunction "Pin_3") (pintype "passive"))
     (pad "4" thru_hole oval locked (at 0 -7.62 180) (size 1.7 1.7) (drill 1) (layers *.Cu *.Mask)
-      (net 17 "/D[17]") (pinfunction "Pin_4") (pintype "passive"))
+      (net 13 "/D17") (pinfunction "Pin_4") (pintype "passive"))
     (pad "5" thru_hole oval locked (at 0 -10.16 180) (size 1.7 1.7) (drill 1) (layers *.Cu *.Mask)
-      (net 16 "/RST{slash}D[16]") (pinfunction "Pin_5") (pintype "passive"))
+      (net 14 "/RST{slash}D16") (pinfunction "Pin_5") (pintype "passive"))
     (pad "6" thru_hole oval locked (at 0 -12.7 180) (size 1.7 1.7) (drill 1) (layers *.Cu *.Mask)
-      (net 15 "/D[15]{slash}SPI.MOSI") (pinfunction "Pin_6") (pintype "passive"))
+      (net 15 "/D15{slash}SPI.MOSI") (pinfunction "Pin_6") (pintype "passive"))
     (pad "7" thru_hole oval locked (at 0 -15.24 180) (size 1.7 1.7) (drill 1) (layers *.Cu *.Mask)
-      (net 14 "/D[14]{slash}SPI.MISO") (pinfunction "Pin_7") (pintype "passive"))
+      (net 16 "/D14{slash}SPI.MISO") (pinfunction "Pin_7") (pintype "passive"))
     (pad "8" thru_hole oval locked (at 0 -17.78 180) (size 1.7 1.7) (drill 1) (layers *.Cu *.Mask)
-      (net 13 "/D[13]{slash}SPI.CS") (pinfunction "Pin_8") (pintype "passive"))
+      (net 17 "/D13{slash}SPI.CS") (pinfunction "Pin_8") (pintype "passive"))
     (pad "9" thru_hole oval locked (at 0 -20.32 180) (size 1.7 1.7) (drill 1) (layers *.Cu *.Mask)
-      (net 12 "/D[12]{slash}SPI.CS") (pinfunction "Pin_9") (pintype "passive"))
+      (net 18 "/D12{slash}SPI.CS") (pinfunction "Pin_9") (pintype "passive"))
     (pad "10" thru_hole oval locked (at 0 -22.86 180) (size 1.7 1.7) (drill 1) (layers *.Cu *.Mask)
-      (net 11 "/D[11]") (pinfunction "Pin_10") (pintype "passive"))
+      (net 19 "/D11") (pinfunction "Pin_10") (pintype "passive"))
     (model "${KICAD6_3DMODEL_DIR}/Connector_PinSocket_2.54mm.3dshapes/PinSocket_1x10_P2.54mm_Vertical.wrl"
       (offset (xyz 0 0 0))
