File: Projects/TI-LaunchPad-BoosterPack-20pin/TI-LaunchPad-BoosterPack-20pin.kicad_sch (KiCad schematic)
At the start: 2 parts, among them J1 Conn_01x10, J2 Conn_01x10

Commit message: Fix v6 net names
Connections:
- net *D[19] renamed *D19
- net D[10]/SDA renamed D10/SDA
- net D[11] renamed D11
- net D[12]/SPI.CS renamed D12/SPI.CS
- net D[13]/SPI.CS renamed D13/SPI.CS
- net D[14]/SPI.MISO renamed D14/SPI.MISO
- net D[15]/SPI.MOSI renamed D15/SPI.MOSI
- net D[17] renamed D17
- net D[18]/SPI.CS renamed D18/SPI.CS
- net D[2]/A renamed D2/A
- net D[3]/UART.RX renamed D3/UART.RX
- net D[4]/UART.TX renamed D4/UART.TX
- net D[5] renamed D5
- net D[6]/A renamed D6/A
- net D[7]/SPI.CLK renamed D7/SPI.CLK
- net D[8] renamed D8
- net D[9]/SCL renamed D9/SCL
- net RST/D[16] renamed RST/D16
Other:
- note added: "Dn pins follow the Energia numbering scheme * PWM-capable pin All pin naming is generic. Exact pin functions vary depending on the LaunchPad, consult the manual."
- note removed: "D[n] pins follow the Energia numbering scheme * PWM-capable pin All pin naming is generic. Exact pin functions vary depending on the LaunchPad, consult the manual."
Changed lines of the file:
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@@
     (stroke (width 0) (type solid) (color 0 0 0 0))
   )
-  (text "D[n] pins follow the Energia numbering scheme\n* PWM-capable pin\n\nAll pin naming is generic. Exact pin functions vary depending on the LaunchPad, consult the manual."
+  (text "Dn pins follow the Energia numbering scheme\n* PWM-capable pin\n\nAll pin naming is generic. Exact pin functions vary depending on the LaunchPad, consult the manual."
     (at 177.8 180.34 0)
     (effects (font (size 1.27 1.27)) (justify left bottom))
   )
-  (label "D[2]{slash}A" (at 25.4 27.94 0)
+  (label "D2{slash}A" (at 25.4 27.94 0)
     (effects (font (size 1.27 1.27)) (justify left bottom))
   )
-  (label "D[11]" (at 88.9 48.26 180)
+  (label "D11" (at 88.9 48.26 180)
     (effects (font (size 1.27 1.27)) (justify right bottom))
   )
-  (label "D[15]{slash}SPI.MOSI" (at 88.9 38.1 180)
+  (label "D15{slash}SPI.MOSI" (at 88.9 38.1 180)
     (effects (font (size 1.27 1.27)) (justify right bottom))
   )
-  (label "D[18]{slash}SPI.CS" (at 88.9 30.48 180)
+  (label "D18{slash}SPI.CS" (at 88.9 30.48 180)
     (effects (font (size 1.27 1.27)) (justify right bottom))
   )
-  (label "D[7]{slash}SPI.CLK" (at 25.4 40.64 0)
+  (label "D7{slash}SPI.CLK" (at 25.4 40.64 0)
     (effects (font (size 1.27 1.27)) (justify left bottom))
   )
-  (label "D[17]" (at 88.9 33.02 180)
+  (label "D17" (at 88.9 33.02 180)
     (effects (font (size 1.27 1.27)) (justify right bottom))
   )
-  (label "D[6]{slash}A" (at 25.4 38.1 0)
+  (label "D6{slash}A" (at 25.4 38.1 0)
     (effects (font (size 1.27 1.27)) (justify left bottom))
   )
-  (label "*D[19]" (at 88.9 27.94 180)
+  (label "*D19" (at 88.9 27.94 180)
     (effects (font (size 1.27 1.27)) (justify right bottom))
   )
-  (label "D[9]{slash}SCL" (at 25.4 45.72 0)
+  (label "D9{slash}SCL" (at 25.4 45.72 0)
     (effects (font (size 1.27 1.27)) (justify left bottom))
   )
-  (label "RST{slash}D[16]" (at 88.9 35.56 180)
+  (label "RST{slash}D16" (at 88.9 35.56 180)
     (effects (font (size 1.27 1.27)) (justify right bottom))
   )
-  (label "D[10]{slash}SDA" (at 25.4 48.26 0)
+  (label "D10{slash}SDA" (at 25.4 48.26 0)
     (effects (font (size 1.27 1.27)) (justify left bottom))
   )
-  (label "D[5]" (at 25.4 35.56 0)
+  (label "D5" (at 25.4 35.56 0)
     (effects (font (size 1.27 1.27)) (justify left bottom))
   )
-  (label "D[13]{slash}SPI.CS" (at 88.9 43.18 180)
+  (label "D13{slash}SPI.CS" (at 88.9 43.18 180)
     (effects (font (size 1.27 1.27)) (justify right bottom))
   )
-  (label "D[4]{slash}UART.TX" (at 25.4 33.02 0)
+  (label "D4{slash}UART.TX" (at 25.4 33.02 0)
     (effects (font (size 1.27 1.27)) (justify left bottom))
   )
-  (label "D[8]" (at 25.4 43.18 0)
+  (label "D8" (at 25.4 43.18 0)
     (effects (font (size 1.27 1.27)) (justify left bottom))
   )
-  (label "D[14]{slash}SPI.MISO" (at 88.9 40.64 180)
+  (label "D14{slash}SPI.MISO" (at 88.9 40.64 180)
     (effects (font (size 1.27 1.27)) (justify right bottom))
   )
-  (label "D[12]{slash}SPI.CS" (at 88.9 45.72 180)
+  (label "D12{slash}SPI.CS" (at 88.9 45.72 180)
     (effects (font (size 1.27 1.27)) (justify right bottom))
   )
-  (label "D[3]{slash}UART.RX" (at 25.4 30.48 0)
+  (label "D3{slash}UART.RX" (at 25.4 30.48 0)
     (effects (font (size 1.27 1.27)) (justify left bottom))
   )
