File: Projects/TI-LaunchPad-BoosterPack-40pin/TI-LaunchPad-BoosterPack-40pin.kicad_sch (KiCad schematic)
At the start: 2 parts, among them J2-J4 Conn_01x10, J3-J1 Conn_01x10

Commit message: Fix v6 net names
Connections:
- net *D[19] renamed *D19
- net *D[37] renamed *D37
- net *D[38] renamed *D38
- net *D[39] renamed *D39
- net *D[40] renamed *D40
- net D[10]/SDA renamed D10/SDA
- net D[11] renamed D11
- net D[12]/SPI.CS renamed D12/SPI.CS
- net D[13]/SPI.CS renamed D13/SPI.CS
- net D[14]/SPI.MISO renamed D14/SPI.MISO
- net D[15]/SPI.MOSI renamed D15/SPI.MOSI
- net D[17] renamed D17
- net D[18]/SPI.CS renamed D18/SPI.CS
- net D[23]/ADC renamed D23/ADC
- net D[24]/ADC renamed D24/ADC
- net D[25]/ADC renamed D25/ADC
- net D[26]/ADC renamed D26/ADC
- net D[27]/ADC renamed D27/ADC
- net D[28]/ADC renamed D28/ADC
- net D[29]/DAC renamed D29/DAC
- net D[2]/ADC renamed D2/ADC
- net D[30]/DAC renamed D30/DAC
- net D[31] renamed D31
- net D[32] renamed D32
- net D[33] renamed D33
- net D[34] renamed D34
- net D[35]/TC renamed D35/TC
- net D[36]/TC renamed D36/TC
- net D[3]/UART.RX renamed D3/UART.RX
- net D[4]/UART.TX renamed D4/UART.TX
- net D[5] renamed D5
- net D[6]/ADC renamed D6/ADC
- net D[7]/SPI.CLK renamed D7/SPI.CLK
- net D[8] renamed D8
- net D[9]/SCL renamed D9/SCL
- net RST/D[16] renamed RST/D16
Other:
- note added: "Dn pins follow the Energia numbering scheme * PWM-capable pin TC: timer capture pin All pin naming is generic. Exact pin functions vary depending on the LaunchPad, consult the manual."
- note removed: "D[n] pins follow the Energia numbering scheme * PWM-capable pin TC: timer capture pin All pin naming is generic. Exact pin functions vary depending on the LaunchPad, consult the manual."
Changed lines of the file:
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@@
     (stroke (width 0) (type solid) (color 0 0 0 0))
   )
-  (text "D[n] pins follow the Energia numbering scheme\n* PWM-capable pin\nTC: timer capture pin\n\nAll pin naming is generic. Exact pin functions vary depending on the LaunchPad, consult the manual."
+  (text "Dn pins follow the Energia numbering scheme\n* PWM-capable pin\nTC: timer capture pin\n\nAll pin naming is generic. Exact pin functions vary depending on the LaunchPad, consult the manual."
     (at 177.8 180.34 0)
     (effects (font (size 1.27 1.27)) (justify left bottom))
   )
-  (label "D[2]{slash}ADC" (at 27.94 27.94 0)
+  (label "D2{slash}ADC" (at 27.94 27.94 0)
     (effects (font (size 1.27 1.27)) (justify left bottom))
   )
-  (label "D[11]" (at 128.27 48.26 180)
+  (label "D11" (at 128.27 48.26 180)
     (effects (font (size 1.27 1.27)) (justify right bottom))
   )
-  (label "*D[38]" (at 78.74 30.48 0)
+  (label "*D38" (at 78.74 30.48 0)
     (effects (font (size 1.27 1.27)) (justify left bottom))
   )
-  (label "D[29]{slash}DAC" (at 73.66 45.72 180)
+  (label "D29{slash}DAC" (at 73.66 45.72 180)
     (effects (font (size 1.27 1.27)) (justify right bottom))
   )
-  (label "D[15]{slash}SPI.MOSI" (at 128.27 38.1 180)
+  (label "D15{slash}SPI.MOSI" (at 128.27 38.1 180)
     (effects (font (size 1.27 1.27)) (justify right bottom))
   )
-  (label "D[25]{slash}ADC" (at 73.66 35.56 180)
+  (label "D25{slash}ADC" (at 73.66 35.56 180)
     (effects (font (size 1.27 1.27)) (justify right bottom))
   )
-  (label "D[18]{slash}SPI.CS" (at 128.27 30.48 180)
+  (label "D18{slash}SPI.CS" (at 128.27 30.48 180)
     (effects (font (size 1.27 1.27)) (justify right bottom))
   )
-  (label "D[31]" (at 78.74 48.26 0)
+  (label "D31" (at 78.74 48.26 0)
     (effects (font (size 1.27 1.27)) (justify left bottom))
   )
-  (label "D[24]{slash}ADC" (at 73.66 33.02 180)
+  (label "D24{slash}ADC" (at 73.66 33.02 180)
     (effects (font (size 1.27 1.27)) (justify right bottom))
   )
-  (label "D[7]{slash}SPI.CLK" (at 27.94 40.64 0)
+  (label "D7{slash}SPI.CLK" (at 27.94 40.64 0)
     (effects (font (size 1.27 1.27)) (justify left bottom))
   )
-  (label "D[33]" (at 78.74 43.18 0)
+  (label "D33" (at 78.74 43.18 0)
     (effects (font (size 1.27 1.27)) (justify left bottom))
   )
-  (label "D[17]" (at 128.27 33.02 180)
+  (label "D17" (at 128.27 33.02 180)
     (effects (font (size 1.27 1.27)) (justify right bottom))
   )
-  (label "D[6]{slash}ADC" (at 27.94 38.1 0)
+  (label "D6{slash}ADC" (at 27.94 38.1 0)
     (effects (font (size 1.27 1.27)) (justify left bottom))
   )
-  (label "*D[19]" (at 128.27 27.94 180)
+  (label "*D19" (at 128.27 27.94 180)
     (effects (font (size 1.27 1.27)) (justify right bottom))
   )
-  (label "D[9]{slash}SCL" (at 27.94 45.72 0)
+  (label "D9{slash}SCL" (at 27.94 45.72 0)
     (effects (font (size 1.27 1.27)) (justify left bottom))
   )
-  (label "RST{slash}D[16]" (at 128.27 35.56 180)
+  (label "RST{slash}D16" (at 128.27 35.56 180)
     (effects (font (size 1.27 1.27)) (justify right bottom))
   )
-  (label "D[35]{slash}TC" (at 78.74 38.1 0)
+  (label "D35{slash}TC" (at 78.74 38.1 0)
     (effects (font (size 1.27 1.27)) (justify left bottom))
   )
-  (label "D[10]{slash}SDA" (at 27.94 48.26 0)
+  (label "D10{slash}SDA" (at 27.94 48.26 0)
     (effects (font (size 1.27 1.27)) (justify left bottom))
   )
-  (label "D[5]" (at 27.94 35.56 0)
+  (label "D5" (at 27.94 35.56 0)
     (effects (font (size 1.27 1.27)) (justify left bottom))
   )
-  (label "D[27]{slash}ADC" (at 73.66 40.64 180)
+  (label "D27{slash}ADC" (at 73.66 40.64 180)
     (effects (font (size 1.27 1.27)) (justify right bottom))
   )
-  (label "D[28]{slash}ADC" (at 73.66 43.18 180)
+  (label "D28{slash}ADC" (at 73.66 43.18 180)
     (effects (font (size 1.27 1.27)) (justify right bottom))
   )
-  (label "D[13]{slash}SPI.CS" (at 128.27 43.18 180)
+  (label "D13{slash}SPI.CS" (at 128.27 43.18 180)
     (effects (font (size 1.27 1.27)) (justify right bottom))
   )
-  (label "D[23]{slash}ADC" (at 73.66 30.48 180)
+  (label "D23{slash}ADC" (at 73.66 30.48 180)
     (effects (font (size 1.27 1.27)) (justify right bottom))
   )
-  (label "*D[39]" (at 78.74 27.94 0)
+  (label "*D39" (at 78.74 27.94 0)
     (effects (font (size 1.27 1.27)) (justify left bottom))
   )
-  (label "*D[40]" (at 78.74 25.4 0)
+  (label "*D40" (at 78.74 25.4 0)
     (effects (font (size 1.27 1.27)) (justify left bottom))
   )
-  (label "D[4]{slash}UART.TX" (at 27.94 33.02 0)
+  (label "D4{slash}UART.TX" (at 27.94 33.02 0)
     (effects (font (size 1.27 1.27)) (justify left bottom))
   )
-  (label "D[8]" (at 27.94 43.18 0)
+  (label "D8" (at 27.94 43.18 0)
     (effects (font (size 1.27 1.27)) (justify left bottom))
   )
-  (label "D[36]{slash}TC" (at 78.74 35.56 0)
+  (label "D36{slash}TC" (at 78.74 35.56 0)
     (effects (font (size 1.27 1.27)) (justify left bottom))
   )
-  (label "D[30]{slash}DAC" (at 73.66 48.26 180)
+  (label "D30{slash}DAC" (at 73.66 48.26 180)
     (effects (font (size 1.27 1.27)) (justify right bottom))
   )
-  (label "D[32]" (at 78.74 45.72 0)
+  (label "D32" (at 78.74 45.72 0)
     (effects (font (size 1.27 1.27)) (justify left bottom))
   )
-  (label "D[34]" (at 78.74 40.64 0)
+  (label "D34" (at 78.74 40.64 0)
     (effects (font (size 1.27 1.27)) (justify left bottom))
   )
-  (label "*D[37]" (at 78.74 33.02 0)
+  (label "*D37" (at 78.74 33.02 0)
     (effects (font (size 1.27 1.27)) (justify left bottom))
   )
-  (label "D[14]{slash}SPI.MISO" (at 128.27 40.64 180)
+  (label "D14{slash}SPI.MISO" (at 128.27 40.64 180)
     (effects (font (size 1.27 1.27)) (justify right bottom))
   )
-  (label "D[12]{slash}SPI.CS" (at 128.27 45.72 180)
+  (label "D12{slash}SPI.CS" (at 128.27 45.72 180)
     (effects (font (size 1.27 1.27)) (justify right bottom))
   )
-  (label "D[3]{slash}UART.RX" (at 27.94 30.48 0)
+  (label "D3{slash}UART.RX" (at 27.94 30.48 0)
     (effects (font (size 1.27 1.27)) (justify left bottom))
   )
-  (label "D[26]{slash}ADC" (at 73.66 38.1 180)
+  (label "D26{slash}ADC" (at 73.66 38.1 180)
     (effects (font (size 1.27 1.27)) (justify right bottom))
   )
