File: Projects/STM32_Nucleo-144_Zio/STM32_Nucleo-144_Zio.kicad_pcb (KiCad board)
At the start: 4 copper layers, 53.6 x 74.2 mm, 4 parts, among them J1 CN8, J2 CN7, J3 CN9, J4 CN10

Commit message: fix extra layers
Parts:
- moved J1 6.54 mm to (120.8, 77.7)
- moved J2 6.54 mm to (166.6, 68.5)
- moved J3 6.54 mm to (120.8, 100.5)
- moved J4 6.54 mm to (166.6, 95.5)
Connections:
- J1 pad 1: unconnected-(J1-Pin_1-Pad1) -> (no net)
- J1 pad 10: unconnected-(J1-Pin_10-Pad10) -> (no net)
- J1 pad 11: GND -> (no net)
- J1 pad 12: unconnected-(J1-Pin_12-Pad12) -> (no net)
- J1 pad 13: GND -> (no net)
- J1 pad 14: unconnected-(J1-Pin_14-Pad14) -> (no net)
- J1 pad 15: /VIN -> (no net)
- J1 pad 16: unconnected-(J1-Pin_16-Pad16) -> (no net)
- J1 pad 2: unconnected-(J1-Pin_2-Pad2) -> (no net)
- J1 pad 3: /IOREF -> (no net)
- J1 pad 4: unconnected-(J1-Pin_4-Pad4) -> (no net)
- J1 pad 5: /~{RST} -> (no net)
- J1 pad 6: unconnected-(J1-Pin_6-Pad6) -> (no net)
- J1 pad 7: +3V3 -> (no net)
- J1 pad 8: unconnected-(J1-Pin_8-Pad8) -> (no net)
- J1 pad 9: +5V -> (no net)
- J2 pad 1: unconnected-(J2-Pin_1-Pad1) -> (no net)
- J2 pad 10: unconnected-(J2-Pin_10-Pad10) -> (no net)
- J2 pad 11: unconnected-(J2-Pin_11-Pad11) -> (no net)
- J2 pad 12: unconnected-(J2-Pin_12-Pad12) -> (no net)
- J2 pad 13: unconnected-(J2-Pin_13-Pad13) -> (no net)
- J2 pad 14: unconnected-(J2-Pin_14-Pad14) -> (no net)
- J2 pad 15: unconnected-(J2-Pin_15-Pad15) -> (no net)
- J2 pad 16: unconnected-(J2-Pin_16-Pad16) -> (no net)
- J2 pad 17: unconnected-(J2-Pin_17-Pad17) -> (no net)
- J2 pad 18: unconnected-(J2-Pin_18-Pad18) -> (no net)
- J2 pad 19: unconnected-(J2-Pin_19-Pad19) -> (no net)
- J2 pad 2: unconnected-(J2-Pin_2-Pad2) -> (no net)
- J2 pad 20: unconnected-(J2-Pin_20-Pad20) -> (no net)
- J2 pad 3: unconnected-(J2-Pin_3-Pad3) -> (no net)
- J2 pad 4: unconnected-(J2-Pin_4-Pad4) -> (no net)
- J2 pad 5: unconnected-(J2-Pin_5-Pad5) -> (no net)
- J2 pad 6: /VREFP -> (no net)
- J2 pad 7: unconnected-(J2-Pin_7-Pad7) -> (no net)
- J2 pad 8: GND -> (no net)
- J2 pad 9: unconnected-(J2-Pin_9-Pad9) -> (no net)
- J3 pad 1: unconnected-(J3-Pin_1-Pad1) -> (no net)
- J3 pad 10: unconnected-(J3-Pin_10-Pad10) -> (no net)
- J3 pad 11: unconnected-(J3-Pin_11-Pad11) -> (no net)
- J3 pad 12: GND -> (no net)
- J3 pad 13: unconnected-(J3-Pin_13-Pad13) -> (no net)
- J3 pad 14: unconnected-(J3-Pin_14-Pad14) -> (no net)
- J3 pad 15: unconnected-(J3-Pin_15-Pad15) -> (no net)
- J3 pad 16: unconnected-(J3-Pin_16-Pad16) -> (no net)
- J3 pad 17: unconnected-(J3-Pin_17-Pad17) -> (no net)
- J3 pad 18: unconnected-(J3-Pin_18-Pad18) -> (no net)
- J3 pad 19: unconnected-(J3-Pin_19-Pad19) -> (no net)
- J3 pad 2: unconnected-(J3-Pin_2-Pad2) -> (no net)
- J3 pad 20: unconnected-(J3-Pin_20-Pad20) -> (no net)
- J3 pad 21: unconnected-(J3-Pin_21-Pad21) -> (no net)
- J3 pad 22: unconnected-(J3-Pin_22-Pad22) -> (no net)
- J3 pad 23: GND -> (no net)
- J3 pad 24: unconnected-(J3-Pin_24-Pad24) -> (no net)
- J3 pad 25: unconnected-(J3-Pin_25-Pad25) -> (no net)
- J3 pad 26: unconnected-(J3-Pin_26-Pad26) -> (no net)
- J3 pad 27: unconnected-(J3-Pin_27-Pad27) -> (no net)
- J3 pad 28: unconnected-(J3-Pin_28-Pad28) -> (no net)
- J3 pad 29: unconnected-(J3-Pin_29-Pad29) -> (no net)
- J3 pad 3: unconnected-(J3-Pin_3-Pad3) -> (no net)
- J3 pad 30: unconnected-(J3-Pin_30-Pad30) -> (no net)
- J3 pad 4: unconnected-(J3-Pin_4-Pad4) -> (no net)
- J3 pad 5: unconnected-(J3-Pin_5-Pad5) -> (no net)
- J3 pad 6: unconnected-(J3-Pin_6-Pad6) -> (no net)
- J3 pad 7: unconnected-(J3-Pin_7-Pad7) -> (no net)
- J3 pad 8: unconnected-(J3-Pin_8-Pad8) -> (no net)
- J3 pad 9: unconnected-(J3-Pin_9-Pad9) -> (no net)
- J4 pad 1: VDDA -> (no net)
- J4 pad 10: unconnected-(J4-Pin_10-Pad10) -> (no net)
- J4 pad 11: unconnected-(J4-Pin_11-Pad11) -> (no net)
- J4 pad 12: unconnected-(J4-Pin_12-Pad12) -> (no net)
- J4 pad 13: unconnected-(J4-Pin_13-Pad13) -> (no net)
- J4 pad 14: unconnected-(J4-Pin_14-Pad14) -> (no net)
- J4 pad 15: unconnected-(J4-Pin_15-Pad15) -> (no net)
- J4 pad 16: unconnected-(J4-Pin_16-Pad16) -> (no net)
- J4 pad 17: GND -> (no net)
- J4 pad 18: unconnected-(J4-Pin_18-Pad18) -> (no net)
- J4 pad 19: unconnected-(J4-Pin_19-Pad19) -> (no net)
- J4 pad 2: unconnected-(J4-Pin_2-Pad2) -> (no net)
- J4 pad 20: unconnected-(J4-Pin_20-Pad20) -> (no net)
- J4 pad 21: unconnected-(J4-Pin_21-Pad21) -> (no net)
- J4 pad 22: GND -> (no net)
- J4 pad 23: unconnected-(J4-Pin_23-Pad23) -> (no net)
- J4 pad 24: unconnected-(J4-Pin_24-Pad24) -> (no net)
- J4 pad 25: unconnected-(J4-Pin_25-Pad25) -> (no net)
- J4 pad 26: unconnected-(J4-Pin_26-Pad26) -> (no net)
- J4 pad 27: GND -> (no net)
- J4 pad 28: unconnected-(J4-Pin_28-Pad28) -> (no net)
- J4 pad 29: unconnected-(J4-Pin_29-Pad29) -> (no net)
- J4 pad 3: GNDA -> (no net)
- J4 pad 30: unconnected-(J4-Pin_30-Pad30) -> (no net)
- J4 pad 31: unconnected-(J4-Pin_31-Pad31) -> (no net)
- J4 pad 32: unconnected-(J4-Pin_32-Pad32) -> (no net)
- J4 pad 33: unconnected-(J4-Pin_33-Pad33) -> (no net)
- J4 pad 34: unconnected-(J4-Pin_34-Pad34) -> (no net)
- J4 pad 4: unconnected-(J4-Pin_4-Pad4) -> (no net)
- J4 pad 5: GND -> (no net)
- J4 pad 6: unconnected-(J4-Pin_6-Pad6) -> (no net)
- J4 pad 7: unconnected-(J4-Pin_7-Pad7) -> (no net)
- J4 pad 8: unconnected-(J4-Pin_8-Pad8) -> (no net)
- J4 pad 9: unconnected-(J4-Pin_9-Pad9) -> (no net)
Routing:
- net (no net): track 2020.8 -> 0.00 mm
Other:
- copper layers 4 -> 2
